File: HDMI_Switch.kicad_sch (KiCad schematic)
At the start: 16 parts, among them U5 HD3SS215RTQR

Commit message: Added series resistors for USB_DET & SW, HubOsc testpoints
Parts:
- added TP5: TestPoint, TestPoint:TestPoint_Pad_D1.0mm, symbol Connector:TestPoint
- renumbered R3 to R2, R4 to R3, R5 to R4, R6 to R5, R7 to R6, R8 to R7, R9 to R8, TP5 to TP16, U5 to U3
Connections:
- net SW: now also TP5.1
Changed lines of the file:
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@@
 	)
 	(junction
+		(at 176.53 132.08)
+		(diameter 0)
+		(color 0 0 0 0)
+	)
+	(junction
 		(at 142.24 33.02)
 		(diameter 0)
@@
 	(wire
 		(pts
-			(xy 158.75 132.08) (xy 181.61 132.08)
+			(xy 158.75 132.08) (xy 176.53 132.08)
 		)
 		(stroke
@@
 	(wire
 		(pts
+			(xy 176.53 132.08) (xy 181.61 132.08)
+		)
+		(stroke
+			(width 0)
+			(type default)
+		)
+	)
+	(wire
+		(pts
 			(xy 67.31 48.26) (xy 71.12 48.26)
 		)
@@
 	(symbol
 		(lib_id "Connector:TestPoint")
+		(at 176.53 132.08 180)
+		(unit 1)
+		(body_style 1)
+		(exclude_from_sim no)
+		(in_bom no)
+		(on_board yes)
+		(in_pos_files yes)
+		(dnp no)
+		(property "Reference" "TP5"
+			(at 176.53 137.414 0)
+			(show_name no)
+			(do_not_autoplace no)
+			(effects
+				(font
+					(size 1.27 1.27)
+				)
+			)
+		)
+		(property "Value" "TestPoint"
+			(at 173.99 135.382 90)
+			(hide yes)
+			(show_name no)
+			(do_not_autoplace no)
+			(effects
+				(font
+					(size 1.27 1.27)
+				)
+			)
+		)
+		(property "Footprint" "TestPoint:TestPoint_Pad_D1.0mm"
+			(at 171.45 132.08 0)
+			(hide yes)
+			(show_name no)
+			(do_not_autoplace no)
+			(effects
+				(font
+					(size 1.27 1.27)
+				)
+			)
+		)
+		(property "Datasheet" ""
+			(at 171.45 132.08 0)
+			(hide yes)
+			(show_name no)
+			(do_not_autoplace no)
+			(effects
+				(font
+					(size 1.27 1.27)
+				)
+			)
+		)
+		(property "Description" "test point"
+			(at 176.53 132.08 0)
+			(hide yes)
+			(show_name no)
+			(do_not_autoplace no)
+			(effects
+				(font
+					(size 1.27 1.27)
+				)
+			)
+		)
+		(pin "1"
+		)
+		(instances
+			(project "KVM_Switch"
+				(path "/94386106-ccd4-487f-b5c5-d52ec3dd59db/6e43926c-16e0-4a92-a7fc-ce5a89c8ce59"
+					(reference "TP5")
+					(unit 1)
+				)
+			)
+		)
+	)
+	(symbol
+		(lib_id "Connector:TestPoint")
 		(at 181.61 96.52 90)
 		(unit 1)
@@
 		(in_pos_files yes)
 		(dnp no)
-		(property "Reference" "TP5"
+		(property "Reference" "TP16"
 			(at 94.996 133.35 90)
 			(show_name no)
@@
 			(project "KVM_Switch"
 				(path "/94386106-ccd4-487f-b5c5-d52ec3dd59db/6e43926c-16e0-4a92-a7fc-ce5a89c8ce59"
-					(reference "TP5")
+					(reference "TP16")
 					(unit 1)
 				)
@@
 		(in_pos_files yes)
 		(dnp no)
-		(property "Reference" "R5"
+		(property "Reference" "R4"
 			(at 95.758 90.932 0)
 			(show_name no)
@@
 			(project "KVM_Switch"
 				(path "/94386106-ccd4-487f-b5c5-d52ec3dd59db/6e43926c-16e0-4a92-a7fc-ce5a89c8ce59"
-					(reference "R5")
+					(reference "R4")
 					(unit 1)
 				)
@@
 		(in_pos_files yes)
 		(dnp no)
-		(property "Reference" "R8"
+		(property "Reference" "R7"
 			(at 170.688 136.398 0)
 			(show_name no)
@@
 			(project "KVM_Switch"
 				(path "/94386106-ccd4-487f-b5c5-d52ec3dd59db/6e43926c-16e0-4a92-a7fc-ce5a89c8ce59"
-					(reference "R8")
+					(reference "R7")
 					(unit 1)
 				)
@@
 		(in_pos_files yes)
 		(dnp no)
-		(property "Reference" "R9"
+		(property "Reference" "R8"
 			(at 95.758 151.892 0)
 			(show_name no)
@@
 			(project "KVM_Switch"
 				(path "/94386106-ccd4-487f-b5c5-d52ec3dd59db/6e43926c-16e0-4a92-a7fc-ce5a89c8ce59"
-					(reference "R9")
+					(reference "R8")
 					(unit 1)
 				)
@@
 		(in_pos_files yes)
 		(dnp no)
-		(property "Reference" "R7"
+		(property "Reference" "R6"
 			(at 186.69 122.428 90)
 			(show_name no)
@@
 			(project "KVM_Switch"
 				(path "/94386106-ccd4-487f-b5c5-d52ec3dd59db/6e43926c-16e0-4a92-a7fc-ce5a89c8ce59"
-					(reference "R7")
+					(reference "R6")
 					(unit 1)
 				)
@@
 		(in_pos_files yes)
 		(dnp no)
-		(property "Reference" "R3"
+		(property "Reference" "R2"
 			(at 168.402 62.484 0)
 			(show_name no)
@@
 			(project "KVM_Switch"
 				(path "/94386106-ccd4-487f-b5c5-d52ec3dd59db/6e43926c-16e0-4a92-a7fc-ce5a89c8ce59"
-					(reference "R3")
+					(reference "R2")
 					(unit 1)
 				)
@@
 		(in_pos_files yes)
 		(dnp no)
-		(property "Reference" "R6"
+		(property "Reference" "R5"
 			(at 176.53 122.428 90)
 			(show_name no)
@@
 			(project "KVM_Switch"
 				(path "/94386106-ccd4-487f-b5c5-d52ec3dd59db/6e43926c-16e0-4a92-a7fc-ce5a89c8ce59"
-					(reference "R6")
+					(reference "R5")
 					(unit 1)
 				)
@@
 		(in_pos_files yes)
 		(dnp no)
-		(property "Reference" "U5"
+		(property "Reference" "U3"
 			(at 143.256 49.022 0)
 			(show_name no)
@@
 			(project "KVM_Switch"
 				(path "/94386106-ccd4-487f-b5c5-d52ec3dd59db/6e43926c-16e0-4a92-a7fc-ce5a89c8ce59"
-					(reference "U5")
+					(reference "U3")
 					(unit 1)
 				)
@@
 		(in_pos_files yes)
 		(dnp no)
-		(property "Reference" "R4"
+		(property "Reference" "R3"
 			(at 174.752 62.484 0)
 			(show_name no)
@@
 			(project "KVM_Switch"
 				(path "/94386106-ccd4-487f-b5c5-d52ec3dd59db/6e43926c-16e0-4a92-a7fc-ce5a89c8ce59"
-					(reference "R4")
+					(reference "R3")
 					(unit 1)
 				)

Commit message: Added ESD protection for the remaining HDMI pins - Not routed yet
Parts:
- renumbered R2 to R3, R3 to R4, R4 to R5, R5 to R6, R6 to R7, R7 to R8, R8 to R9, TP16 to TP6, U3 to U10
Changed lines of the file:
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@@
 		(in_pos_files yes)
 		(dnp no)
-		(property "Reference" "#PWR07"
+		(property "Reference" "#PWR013"
 			(at 142.24 33.02 0)
 			(hide yes)
@@
 			(project "KVM_Switch"
 				(path "/94386106-ccd4-487f-b5c5-d52ec3dd59db/6e43926c-16e0-4a92-a7fc-ce5a89c8ce59"
-					(reference "#PWR07")
+					(reference "#PWR013")
 					(unit 1)
 				)
@@
 		(in_pos_files yes)
 		(dnp no)
-		(property "Reference" "#PWR014"
+		(property "Reference" "#PWR020"
 			(at 191.77 132.08 0)
 			(hide yes)
@@
 			(project "KVM_Switch"
 				(path "/94386106-ccd4-487f-b5c5-d52ec3dd59db/6e43926c-16e0-4a92-a7fc-ce5a89c8ce59"
-					(reference "#PWR014")
+					(reference "#PWR020")
 					(unit 1)
 				)
@@
 		(in_pos_files yes)
 		(dnp no)
-		(property "Reference" "#PWR016"
+		(property "Reference" "#PWR022"
 			(at 167.64 148.59 0)
 			(hide yes)
@@
 			(project "KVM_Switch"
 				(path "/94386106-ccd4-487f-b5c5-d52ec3dd59db/6e43926c-16e0-4a92-a7fc-ce5a89c8ce59"
-					(reference "#PWR016")
+					(reference "#PWR022")
 					(unit 1)
 				)
@@
 		(in_pos_files yes)
 		(dnp no)
-		(property "Reference" "#PWR011"
+		(property "Reference" "#PWR017"
 			(at 199.39 87.63 0)
 			(hide yes)
@@
 			(project "KVM_Switch"
 				(path "/94386106-ccd4-487f-b5c5-d52ec3dd59db/6e43926c-16e0-4a92-a7fc-ce5a89c8ce59"
-					(reference "#PWR011")
+					(reference "#PWR017")
 					(unit 1)
 				)
@@
 		(in_pos_files yes)
 		(dnp no)
-		(property "Reference" "#PWR09"
+		(property "Reference" "#PWR015"
 			(at 171.45 59.69 0)
 			(hide yes)
@@
 			(project "KVM_Switch"
 				(path "/94386106-ccd4-487f-b5c5-d52ec3dd59db/6e43926c-16e0-4a92-a7fc-ce5a89c8ce59"
-					(reference "#PWR09")
+					(reference "#PWR015")
 					(unit 1)
 				)
@@
 		(in_pos_files yes)
 		(dnp no)
-		(property "Reference" "#PWR015"
+		(property "Reference" "#PWR021"
 			(at 138.43 148.59 0)
 			(hide yes)
@@
 			(project "KVM_Switch"
 				(path "/94386106-ccd4-487f-b5c5-d52ec3dd59db/6e43926c-16e0-4a92-a7fc-ce5a89c8ce59"
-					(reference "#PWR015")
+					(reference "#PWR021")
 					(unit 1)
 				)
@@
 		(in_pos_files yes)
 		(dnp no)
-		(property "Reference" "#PWR017"
+		(property "Reference" "#PWR023"
 			(at 92.71 163.83 0)
 			(hide yes)
@@
 			(project "KVM_Switch"
 				(path "/94386106-ccd4-487f-b5c5-d52ec3dd59db/6e43926c-16e0-4a92-a7fc-ce5a89c8ce59"
-					(reference "#PWR017")
+					(reference "#PWR023")
 					(unit 1)
 				)
@@
 		(in_pos_files yes)
 		(dnp no)
-		(property "Reference" "TP16"
+		(property "Reference" "TP6"
 			(at 94.996 133.35 90)
 			(show_name no)
@@
 			(project "KVM_Switch"
 				(path "/94386106-ccd4-487f-b5c5-d52ec3dd59db/6e43926c-16e0-4a92-a7fc-ce5a89c8ce59"
-					(reference "TP16")
+					(reference "TP6")
 					(unit 1)
 				)
@@
 		(in_pos_files yes)
 		(dnp no)
-		(property "Reference" "R4"
+		(property "Reference" "R5"
 			(at 95.758 90.932 0)
 			(show_name no)
@@
 			(project "KVM_Switch"
 				(path "/94386106-ccd4-487f-b5c5-d52ec3dd59db/6e43926c-16e0-4a92-a7fc-ce5a89c8ce59"
-					(reference "R4")
+					(reference "R5")
 					(unit 1)
 				)
@@
 		(in_pos_files yes)
 		(dnp no)
-		(property "Reference" "R7"
+		(property "Reference" "R8"
 			(at 170.688 136.398 0)
 			(show_name no)
@@
 			(project "KVM_Switch"
 				(path "/94386106-ccd4-487f-b5c5-d52ec3dd59db/6e43926c-16e0-4a92-a7fc-ce5a89c8ce59"
-					(reference "R7")
+					(reference "R8")
 					(unit 1)
 				)
@@
 		(in_pos_files yes)
 		(dnp no)
-		(property "Reference" "#PWR08"
+		(property "Reference" "#PWR014"
 			(at 128.27 49.53 0)
 			(hide yes)
@@
 			(project "KVM_Switch"
 				(path "/94386106-ccd4-487f-b5c5-d52ec3dd59db/6e43926c-16e0-4a92-a7fc-ce5a89c8ce59"
-					(reference "#PWR08")
+					(reference "#PWR014")
 					(unit 1)
 				)
@@
 		(in_pos_files yes)
 		(dnp no)
-		(property "Reference" "R8"
+		(property "Reference" "R9"
 			(at 95.758 151.892 0)
 			(show_name no)
@@
 			(project "KVM_Switch"
 				(path "/94386106-ccd4-487f-b5c5-d52ec3dd59db/6e43926c-16e0-4a92-a7fc-ce5a89c8ce59"
-					(reference "R8")
+					(reference "R9")
 					(unit 1)
 				)
@@
 		(in_pos_files yes)
 		(dnp no)
-		(property "Reference" "R6"
+		(property "Reference" "R7"
 			(at 186.69 122.428 90)
 			(show_name no)
@@
 			(project "KVM_Switch"
 				(path "/94386106-ccd4-487f-b5c5-d52ec3dd59db/6e43926c-16e0-4a92-a7fc-ce5a89c8ce59"
-					(reference "R6")
+					(reference "R7")
 					(unit 1)
 				)
@@
 		(in_pos_files yes)
 		(dnp no)
-		(property "Reference" "#PWR010"
+		(property "Reference" "#PWR016"
 			(at 199.39 71.12 0)
 			(hide yes)
@@
 			(project "KVM_Switch"
 				(path "/94386106-ccd4-487f-b5c5-d52ec3dd59db/6e43926c-16e0-4a92-a7fc-ce5a89c8ce59"
-					(reference "#PWR010")
+					(reference "#PWR016")
 					(unit 1)
 				)
@@
 		(in_pos_files yes)
 		(dnp no)
-		(property "Reference" "#PWR013"
+		(property "Reference" "#PWR019"
 			(at 167.64 125.73 0)
 			(hide yes)
@@
 			(project "KVM_Switch"
 				(path "/94386106-ccd4-487f-b5c5-d52ec3dd59db/6e43926c-16e0-4a92-a7fc-ce5a89c8ce59"
-					(reference "#PWR013")
+					(reference "#PWR019")
 					(unit 1)
 				)
@@
 		(in_pos_files yes)
 		(dnp no)
-		(property "Reference" "R2"
+		(property "Reference" "R3"
 			(at 168.402 62.484 0)
 			(show_name no)
@@
 			(project "KVM_Switch"
 				(path "/94386106-ccd4-487f-b5c5-d52ec3dd59db/6e43926c-16e0-4a92-a7fc-ce5a89c8ce59"
-					(reference "R2")
+					(reference "R3")
 					(unit 1)
 				)
@@
 		(in_pos_files yes)
 		(dnp no)
-		(property "Reference" "#PWR012"
+		(property "Reference" "#PWR018"
 			(at 92.71 102.87 0)
 			(hide yes)
@@
 			(project "KVM_Switch"
 				(path "/94386106-ccd4-487f-b5c5-d52ec3dd59db/6e43926c-16e0-4a92-a7fc-ce5a89c8ce59"
-					(reference "#PWR012")
+					(reference "#PWR018")
 					(unit 1)
 				)
@@
 		(in_pos_files yes)
 		(dnp no)
-		(property "Reference" "R5"
+		(property "Reference" "R6"
 			(at 176.53 122.428 90)
 			(show_name no)
@@
 			(project "KVM_Switch"
 				(path "/94386106-ccd4-487f-b5c5-d52ec3dd59db/6e43926c-16e0-4a92-a7fc-ce5a89c8ce59"
-					(reference "R5")
+					(reference "R6")
 					(unit 1)
 				)
@@
 		(in_pos_files yes)
 		(dnp no)
-		(property "Reference" "U3"
+		(property "Reference" "U10"
 			(at 143.256 49.022 0)
 			(show_name no)
@@
 			(project "KVM_Switch"
 				(path "/94386106-ccd4-487f-b5c5-d52ec3dd59db/6e43926c-16e0-4a92-a7fc-ce5a89c8ce59"
-					(reference "U3")
+					(reference "U10")
 					(unit 1)
 				)
@@
 		(in_pos_files yes)
 		(dnp no)
-		(property "Reference" "R3"
+		(property "Reference" "R4"
 			(at 174.752 62.484 0)
 			(show_name no)
@@
 			(project "KVM_Switch"
 				(path "/94386106-ccd4-487f-b5c5-d52ec3dd59db/6e43926c-16e0-4a92-a7fc-ce5a89c8ce59"
-					(reference "R3")
-					(unit 1)
-				)
+					(reference "R4")
+					(unit 1)
+				)

Commit message: Fix naming typo: KVM_Swtich -> KVM_Switch
Renamed the footprint library folder library/KVM_Swtich.pretty to
library/KVM_Switch.pretty and the 3D model swtich_smd_6x6mm.step to
switch_smd_6x6mm.step, and updated every reference across
fp-lib-table, sym-lib-table, the schematics, symbols.kicad_sym, and
the PCB. Also fixed a stray "Swtich A to C" text label.
Parts:
- U10: symbol KVM_Swtich:HD3SS215RTQR -> KVM_Switch:HD3SS215RTQR
Other:
- note added: "Dx_SEL LOW => Switch A to C"
- note removed: "Dx_SEL LOW => Swtich A to C"
Changed lines of the file:
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@@
 		(company "Stanisław Basiuk")
 	)
-	(text "Dx_SEL LOW => Swtich A to C"
+	(text "Dx_SEL LOW => Switch A to C"
 		(exclude_from_sim no)
 		(at 195.072 136.398 0)
@@
 	)
 	(symbol
-		(lib_id "KVM_Swtich:HD3SS215RTQR")
+		(lib_id "KVM_Switch:HD3SS215RTQR")
 		(at 138.43 95.25 0)
 		(unit 1)
