File: USB_Host_Select.kicad_sch (KiCad schematic)
At the start: 13 parts, among them J1 USB_C_Receptacle_USB2.0_16P, J2 USB_C_Receptacle_USB2.0_16P, U1 USBLC6-2SC6, U2 TS3USB221AQRSERQ1, U3 USBLC6-2SC6

Commit message: More schematics fixes & Layout attempt
Parts:
- added R18: 10k, Resistor_SMD:R_0402_1005Metric, symbol Device:R
- U11: renamed from U2; symbol Symbols:TS3USB221AQRSERQ1 -> KVM_Swtich:TS3USB221AQRSERQ1
- renumbered C1 to C13, C2 to C14, C3 to C15, J1 to J5, J2 to J6, R1 to R16, R2 to R17, R3 to R19, R5 to R20, R6 to R21, U1 to U10, U3 to U12
Connections:
- net GND: now also R18.2
- net SW: now also R18.1
- net USB_A_DN: now also U11.1 (1D+); no longer U11.2 (1D-)
- net USB_A_DP: now also U11.2 (1D-); no longer U11.1 (1D+)
- net USB_B_DN: now also U11.3 (2D+); no longer U11.4 (2D-)
- net USB_B_DP: now also U11.4 (2D-); no longer U11.3 (2D+)
- net USB_UP_DN: now also U11.8 (D+); no longer U11.7 (D-)
- net USB_UP_DP: now also U11.7 (D-); no longer U11.8 (D+)
Other:
- note added: "Intentionally swapped D+ with D-"
- company: (none) -> Stanisław Basiuk
- title: (none) -> KVM_Switch

Commit message: Added series resistors for USB_DET & SW, HubOsc testpoints
Parts:
- added R16, R21: 10k, Resistor_SMD:R_0402_1005Metric, symbol Device:R
- added TP15: TestPoint, TestPoint:TestPoint_Pad_D1.0mm, symbol Connector:TestPoint
- renumbered R16 to R17, R17 to R18, R18 to R19, R19 to R20, R20 to R29, R21 to R30
Connections:
- net DET_USB_A: now also R16.2; no longer C13.1, J5.A4 (VBUS), J5.A9 (VBUS), J5.B4 (VBUS), J5.B9 (VBUS), U10.5 (VBUS)
- net DET_USB_B: now also R21.2; no longer C15.1, J6.A4 (VBUS), J6.A9 (VBUS), J6.B4 (VBUS), J6.B9 (VBUS), U12.5 (VBUS)
- net SW: now also TP15.1
- new net: C15.1, J6.A4 (VBUS), J6.A9 (VBUS), J6.B4 (VBUS), J6.B9 (VBUS), R21.1, U12.5 (VBUS)
- new net: C13.1, J5.A4 (VBUS), J5.A9 (VBUS), J5.B4 (VBUS), J5.B9 (VBUS), R16.1, U10.5 (VBUS)

Commit message: Added ESD protection for the remaining HDMI pins - Not routed yet
Parts:
- renumbered R29 to R22, R30 to R23, TP15 to TP16, U10 to U13, U11 to U14, U12 to U15
Changed lines of the file:
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@@
 		(dnp no)
 		(fields_autoplaced yes)
-		(property "Reference" "#PWR040"
+		(property "Reference" "#PWR046"
 			(at 88.9 132.08 0)
 			(hide yes)
@@
 			(project "KVM_Switch"
 				(path "/94386106-ccd4-487f-b5c5-d52ec3dd59db/e397aa06-0b86-4196-a73c-4d06e82b65f2"
-					(reference "#PWR040")
+					(reference "#PWR046")
 					(unit 1)
 				)
@@
 		(in_pos_files yes)
 		(dnp no)
-		(property "Reference" "U12"
+		(property "Reference" "U15"
 			(at 98.552 127.508 0)
 			(show_name no)
@@
 			(project "KVM_Switch"
 				(path "/94386106-ccd4-487f-b5c5-d52ec3dd59db/e397aa06-0b86-4196-a73c-4d06e82b65f2"
-					(reference "U12")
+					(reference "U15")
 					(unit 1)
 				)
@@
 		(dnp no)
 		(fields_autoplaced yes)
-		(property "Reference" "#PWR037"
+		(property "Reference" "#PWR043"
 			(at 160.02 95.25 0)
 			(hide yes)
@@
 			(project "KVM_Switch"
 				(path "/94386106-ccd4-487f-b5c5-d52ec3dd59db/e397aa06-0b86-4196-a73c-4d06e82b65f2"
-					(reference "#PWR037")
+					(reference "#PWR043")
 					(unit 1)
 				)
@@
 		(dnp no)
 		(fields_autoplaced yes)
-		(property "Reference" "#PWR042"
+		(property "Reference" "#PWR048"
 			(at 97.79 146.05 0)
 			(hide yes)
@@
 			(project "KVM_Switch"
 				(path "/94386106-ccd4-487f-b5c5-d52ec3dd59db/e397aa06-0b86-4196-a73c-4d06e82b65f2"
-					(reference "#PWR042")
+					(reference "#PWR048")
 					(unit 1)
 				)
@@
 		(in_pos_files yes)
 		(dnp no)
-		(property "Reference" "R30"
+		(property "Reference" "R23"
 			(at 81.28 128.27 90)
 			(show_name no)
@@
 			(project "KVM_Switch"
 				(path "/94386106-ccd4-487f-b5c5-d52ec3dd59db/e397aa06-0b86-4196-a73c-4d06e82b65f2"
-					(reference "R30")
+					(reference "R23")
 					(unit 1)
 				)
@@
 		(dnp no)
 		(fields_autoplaced yes)
-		(property "Reference" "#PWR041"
+		(property "Reference" "#PWR047"
 			(at 107.95 132.08 0)
 			(hide yes)
@@
 			(project "KVM_Switch"
 				(path "/94386106-ccd4-487f-b5c5-d52ec3dd59db/e397aa06-0b86-4196-a73c-4d06e82b65f2"
-					(reference "#PWR041")
+					(reference "#PWR047")
 					(unit 1)
 				)
@@
 		(in_pos_files yes)
 		(dnp no)
-		(property "Reference" "U10"
+		(property "Reference" "U13"
 			(at 98.552 64.008 0)
 			(show_name no)
@@
 			(project "KVM_Switch"
 				(path "/94386106-ccd4-487f-b5c5-d52ec3dd59db/e397aa06-0b86-4196-a73c-4d06e82b65f2"
-					(reference "U10")
+					(reference "U13")
 					(unit 1)
 				)
@@
 		(dnp no)
 		(fields_autoplaced yes)
-		(property "Reference" "#PWR043"
+		(property "Reference" "#PWR049"
 			(at 60.96 163.83 0)
 			(hide yes)
@@
 			(project "KVM_Switch"
 				(path "/94386106-ccd4-487f-b5c5-d52ec3dd59db/e397aa06-0b86-4196-a73c-4d06e82b65f2"
-					(reference "#PWR043")
+					(reference "#PWR049")
 					(unit 1)
 				)
@@
 		(in_pos_files yes)
 		(dnp no)
-		(property "Reference" "TP15"
+		(property "Reference" "TP16"
 			(at 180.34 106.934 0)
 			(show_name no)
@@
 			(project "KVM_Switch"
 				(path "/94386106-ccd4-487f-b5c5-d52ec3dd59db/e397aa06-0b86-4196-a73c-4d06e82b65f2"
-					(reference "TP15")
+					(reference "TP16")
 					(unit 1)
 				)
@@
 		(in_pos_files yes)
 		(dnp no)
-		(property "Reference" "R29"
+		(property "Reference" "R22"
 			(at 81.28 118.11 90)
 			(show_name no)
@@
 			(project "KVM_Switch"
 				(path "/94386106-ccd4-487f-b5c5-d52ec3dd59db/e397aa06-0b86-4196-a73c-4d06e82b65f2"
-					(reference "R29")
+					(reference "R22")
 					(unit 1)
 				)
@@
 		(in_pos_files yes)
 		(dnp no)
-		(property "Reference" "#PWR036"
+		(property "Reference" "#PWR042"
 			(at 165.1 82.55 0)
 			(hide yes)
@@
 			(project "KVM_Switch"
 				(path "/94386106-ccd4-487f-b5c5-d52ec3dd59db/e397aa06-0b86-4196-a73c-4d06e82b65f2"
-					(reference "#PWR036")
+					(reference "#PWR042")
 					(unit 1)
 				)
@@
 		(dnp no)
 		(fields_autoplaced yes)
-		(property "Reference" "#PWR035"
+		(property "Reference" "#PWR041"
 			(at 97.79 82.55 0)
 			(hide yes)
@@
 			(project "KVM_Switch"
 				(path "/94386106-ccd4-487f-b5c5-d52ec3dd59db/e397aa06-0b86-4196-a73c-4d06e82b65f2"
-					(reference "#PWR035")
+					(reference "#PWR041")
 					(unit 1)
 				)
@@
 		(dnp no)
 		(fields_autoplaced yes)
-		(property "Reference" "#PWR039"
+		(property "Reference" "#PWR045"
 			(at 165.1 121.92 0)
 			(hide yes)
@@
 			(project "KVM_Switch"
 				(path "/94386106-ccd4-487f-b5c5-d52ec3dd59db/e397aa06-0b86-4196-a73c-4d06e82b65f2"
-					(reference "#PWR039")
+					(reference "#PWR045")
 					(unit 1)
 				)
@@
 		(dnp no)
 		(fields_autoplaced yes)
-		(property "Reference" "U11"
+		(property "Reference" "U14"
 			(at 167.2433 88.9 0)
 			(show_name no)
@@
 			(project "KVM_Switch"
 				(path "/94386106-ccd4-487f-b5c5-d52ec3dd59db/e397aa06-0b86-4196-a73c-4d06e82b65f2"
-					(reference "U11")
+					(reference "U14")
 					(unit 1)
 				)
@@
 		(dnp no)
 		(fields_autoplaced yes)
-		(property "Reference" "#PWR033"
+		(property "Reference" "#PWR039"
 			(at 88.9 68.58 0)
 			(hide yes)
@@
 			(project "KVM_Switch"
 				(path "/94386106-ccd4-487f-b5c5-d52ec3dd59db/e397aa06-0b86-4196-a73c-4d06e82b65f2"
-					(reference "#PWR033")
+					(reference "#PWR039")
 					(unit 1)
 				)
@@
 		(dnp no)
 		(fields_autoplaced yes)
-		(property "Reference" "#PWR038"
+		(property "Reference" "#PWR044"
 			(at 60.96 100.33 0)
 			(hide yes)
@@
 			(project "KVM_Switch"
 				(path "/94386106-ccd4-487f-b5c5-d52ec3dd59db/e397aa06-0b86-4196-a73c-4d06e82b65f2"
-					(reference "#PWR038")
+					(reference "#PWR044")
 					(unit 1)
 				)
@@
 		(dnp no)
 		(fields_autoplaced yes)
-		(property "Reference" "#PWR034"
+		(property "Reference" "#PWR040"
 			(at 107.95 68.58 0)
 			(hide yes)
@@
 			(project "KVM_Switch"
 				(path "/94386106-ccd4-487f-b5c5-d52ec3dd59db/e397aa06-0b86-4196-a73c-4d06e82b65f2"
-					(reference "#PWR034")
-					(unit 1)
-				)
+					(reference "#PWR040")
+					(unit 1)
+				)

Commit message: Fix naming typo: KVM_Swtich -> KVM_Switch
Renamed the footprint library folder library/KVM_Swtich.pretty to
library/KVM_Switch.pretty and the 3D model swtich_smd_6x6mm.step to
switch_smd_6x6mm.step, and updated every reference across
fp-lib-table, sym-lib-table, the schematics, symbols.kicad_sym, and
the PCB. Also fixed a stray "Swtich A to C" text label.
Parts:
- U14: footprint KVM_Swtich:TS3USB221AQRSERQ1 -> KVM_Switch:TS3USB221AQRSERQ1; symbol KVM_Swtich:TS3USB221AQRSERQ1 -> KVM_Switch:TS3USB221AQRSERQ1
Changed lines of the file:
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@@
 	)
 	(symbol
-		(lib_id "KVM_Swtich:TS3USB221AQRSERQ1")
+		(lib_id "KVM_Switch:TS3USB221AQRSERQ1")
 		(at 165.1 101.6 0)
 		(unit 1)
@@
 			)
 		)
-		(property "Footprint" "KVM_Swtich:TS3USB221AQRSERQ1"
+		(property "Footprint" "KVM_Switch:TS3USB221AQRSERQ1"
 			(at 165.1 101.6 0)
 			(hide yes)
